Commit message: Full Body Global Compliance

File: model/terrain/pegboard/pegboard17.urdf (robot description, URDF)
Before this commit: robot flat_plane15_15, 1 links, 0 joints
Links:
- removed link flatPlaneLink
- added link peg1, mass .0; collision cylinder length=0.3 radius=0.03; visual cylinder length=0.3 radius=0.03
