Commit message: Decentralized Compliance Added

File: model/terrain/plate3.urdf (robot description, URDF)
Before this commit: robot plate2, 1 links, 0 joints
Links:
- removed link plateLink2
- added link plateLink1, mass .0; collision box size=0.5 0.2 0.5; visual box size=0.5 0.2 0.5

File: model/terrain/plate4.urdf (robot description, URDF)
Before this commit: robot plate2, 1 links, 0 joints
Links:
- removed link plateLink2
- added link plateLink1, mass .0; collision box size=0.5 0.2 0.5; visual box size=0.5 0.2 0.5

File: model/terrain/plate5.urdf (robot description, URDF)
Before this commit: robot plate2, 1 links, 0 joints
Links:
- removed link plateLink2
- added link plateLink1, mass .0; collision box size=0.1 0.08 0.5; visual box size=0.1 0.08 0.5
